File: hardware/MainBoard/MainBoard.kicad_pcb (KiCad board)
At the start: 2 copper layers, 50 x 80 mm, 34 parts, among them J101 Servo, J102 Relay, J103 MotorDriver, J104 MPU9250, J105 PicoBATT+, J106 Tachometer, J201 Micro_SD_Card, J202 Stop, SW101 Reset, SW102 SW_Pico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

Commit message: 発注！
Parts:
- moved G*** 1.23 mm to (158.6, 98.2)
Other:
- board text added: "WASA_Rockoon_2026 CMG_MainBoard_DevModel"
- board text removed: "WASA_Rockoon_2026 CMG_MainBoard"
Changed lines of the file:
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@@
 	(footprint "Library:wasa_10mm"
 		(layer "B.Cu")
-		(at 158.3 97 90)
+		(at 158.59 98.195 90)
 		(property "Reference" "G***"
 			(at 0.108168 -3.048 90)
@@
 		)
 	)
-	(gr_text "WASA_Rockoon_2026\nCMG_MainBoard"
-		(at 152.9 110.2 270)
+	(gr_text "WASA_Rockoon_2026\nCMG_MainBoard_DevModel"
+		(at 151.7 110.2 270)
 		(layer "B.SilkS")
 		(effects

Commit message: 配線ミスを直した
Parts:
- C203: value 0.1 -> 0.1uF
- R204: value All 10k -> 10k
Connections:
- A101 pad 22: /CLK -> /CS
- A101 pad 24: /MOSI -> /CLK
- A101 pad 25: /CS -> /MOSI
Routing:
- net /CLK: track 22.9 -> 28.0 mm
- net /CS: track 51.0 -> 46.0 mm, vias 1 -> 2
- net /MOSI: track 25.1 -> 26.6 mm
