File: hardware/MainBoard/MainBoard.kicad_sch (KiCad schematic)
At the start: 23 parts, among them J101 Servo, J102 Relay, J103 MotorDriver, J104 MPU9250, J105 PicoBATT+, J106 Tachometer, J202 Stop, SW101 Reset, SW102 SW_Pico, SW103 SW_BATT

Commit message: KiCad10で保存
Parts:
- B101: value ~ -> (none)
Connections:
- net CLK: now also A101.24 (GPIO18); no longer A101.22 (GPIO17)
- net CS: now also A101.22 (GPIO17); no longer A101.25 (GPIO19)
- net MOSI: now also A101.25 (GPIO19); no longer A101.24 (GPIO18)
